Commit message: Phase 1: motor 57HSE3.0N -> 57HSE1.5N, still open loop
Holding torque drops 3.0 -> 1.5 N.m. Deliberately landed on its own,
before the closed-loop change, because the two move the system in
opposite directions and mixing them makes the results unreadable.

Open-loop series stiffness K = 1/(1/(Th*Nr) + 1/k):
  azimuth  137.14 -> 71.64 N.m/rad, f_n 4.79 -> 3.46 Hz, zeta 0.0220 -> 0.0304
  tilt     101.82 -> 60.65 N.m/rad, f_n 6.89 -> 5.32 Hz, zeta 0.0425 -> 0.0551

So on the open-loop baseline a weaker motor makes the system softer and
BETTER damped. The closed-loop change in the next phases does the
opposite.

build_model.py carried a hardcoded effort="3" on the elevation joint
that was not derived from Th, unlike cmd_max. It would have survived the
change silently. Now derived.

wind_node selftest pins K to 71.64 / 60.65. The literal pin is kept
deliberately: it caught exactly this class of change.

Regenerated URDF diff is exactly four values: effort 3 -> 1.5, and
p_gain / cmd_max on both joints. All three node selftests pass.

Torque budget consequence, to be addressed in the sizing phase: peak
gravity on the tilt axis is 1.274 N.m, now 85 % of holding torque
instead of 42 %.

File: solar_tracker/solar_tracker.urdf (robot description, URDF)
Before this commit: robot solar_tracker, 9 links, 8 joints
Joints:
- joint elevation_joint: limit lower=-0.7854 upper=0.7854 effort=3 velocity=1 -> lower=-0.7854 upper=0.7854 effort=1.5 velocity=1

File: solar_tracker/solar_tracker_stepper.urdf (robot description, URDF)
Before this commit: robot solar_tracker, 9 links, 8 joints
Joints:
- joint elevation_joint: limit lower=-0.7854 upper=0.7854 effort=3 velocity=1 -> lower=-0.7854 upper=0.7854 effort=1.5 velocity=1
