Commit message: Migrate all nodes to v2 and delete v1
v1 is gone: solar_tracker/ removed entirely. Sun, sensor, EKF, wind,
stepper, both control panels and all four recorders now live in
solar_tracker_v2/. They needed no path edits because every one of them
resolves ROOT as parent.parent, which is still the project root.

dyn_model.AXES IS now the new design, so every node that reads D.AXES
picks it up with no edit. The old direct-drive values are archived as
AXES_V1 for comparison; nothing uses them.

  tilt     N=5.25  k=163.8  K_ser=151.77  Th_L=7.875 N.m  f_n=8.09 Hz
  azimuth  N=1.00  k=1600   K_ser=71.64   Th_L=1.500 N.m  f_n=3.46 Hz

k on tilt corrected 317 -> 163.8: the as_8mm shaft measures 194 mm in
the CAD, not the 100 mm previously assumed. G*J/L for 8 mm steel gives
163.8.

ROS topic names deliberately unchanged (/solar_tracker/*, /sun/state,
/tracker/diag, /ekf/state, /wind/state); only the Gazebo model name
differs, so every existing tool still applies.

TWO REAL PROBLEMS FOUND AND FIXED:

1. The +-170 degree azimuth limit I invented stopped the tracker
   following the sun. Gazebo showed the joint pinned at -170 while the
   sun commanded -178.9, and the EKF then reported NIS 126 against a
   gate of 25. Sweeping 2026 shows q1 actually needs -180.9 to +174.6
   degrees, so even +-180 is short. Set to +-185, still an ASSUMPTION
   pending the real travel from the CAD.

2. The open-loop stepper torque law is no longer valid on a geared
   axis. It needs k > Th_L*Nr_L; the gear raises the load-referred
   magnetic spring to 2067 N.m/rad against a 163.8 shaft, so the
   quasi-static curve becomes multivalued and the bisection cannot pick
   a branch. stepper_node now has sumbu_sah(), skips such axes in
   selftest and logs an error at startup instead of returning silently
   wrong torque. Actuator mode is pid only for this design, which is
   what every Gazebo validation has used anyway.

Verified running headless with sun_node and ekf: 18 topics up, zero
errors in the log, pointing command error 1.09 deg, LDR, single-diode
electrical model, wind and oscillation statistics all publishing.

Still legacy and now orphaned: build_model.py and inersia/ still build
from the old parts_v2 CAD. build_model.py is kept only because
inersia/inersia_cad.py imports it.

File: solar_tracker_v2/solar_tracker_v2.urdf (robot description, URDF)
Before this commit: robot solar_tracker_v2, 4 links, 3 joints
Joints:
- joint azimuth_joint: limit lower=-2.9671 upper=2.9671 effort=1.500 velocity=1 -> lower=-3.2289 upper=3.2289 effort=1.500 velocity=1

Commit message: Correct gear ratio to 5.00:1, measured on the rig
User counted 5 pinion turns per 1 turn of the large gear, and measured
outer diameters 22 and 88 mm. That is the authoritative measurement and
it overrides my CAD-derived figure.

My 5.25:1 was wrong. It came from fitting module 2 with z=8/42 to the
mesh centre distance, and it predicted a 20 mm pinion against the 22 mm
actually fitted.

The measurements reconcile as outer diameters: OD = m(z+2) with
z2/z1 = 5 gives (5*z1+2)/(z1+2) = 88/22 = 4, so z1=6, z2=30, module
2.75. Check: 2.75*8 = 22 and 2.75*32 = 88, both exact. Pitch diameters
16.5 and 82.5, whose ratio is exactly 5. Centre distance 49.5 mm
against 50.2 measured in CAD.

Also wrong: my claim that the large gear is a sector. It is a full
circle, proven by the pinion completing 5 whole turns against it. That
claim rested only on the mesh bounding box being 87.9 x 72.3 rather
than square; my angular-coverage test was unreliable (it flagged the
pinion as a sector too).

Tilt axis now:
  N=5.00  K_ser=150.64  Th_L=7.500 N.m  f_n=8.06 Hz  zeta=0.0336
  microstep at load 0.0225 deg, torque budget 24.0 % of motor holding
  torque, gravity alone 11.8 %

wind_node's pinned tripwire caught the change, which is what it is for.
All four selftests pass and the URDF is regenerated.

File: solar_tracker_v2/solar_tracker_v2.urdf (robot description, URDF)
Before this commit: robot solar_tracker_v2, 4 links, 3 joints
Joints:
- joint elevation_joint: limit lower=-0.7854 upper=0.7854 effort=7.875 velocity=1 -> lower=-0.7854 upper=0.7854 effort=7.500 velocity=1
